File: mcu.kicad_sch (KiCad schematic)
At the start: 39 parts, among them U400 STM32H563VGTx, X300 Q13FC1350000400, Y400 ASE-xxxMHz

Commit message: Change backplane connector arrangement
Parts:
- FB401: value ~ -> (none)
Changed lines of the file:
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@@
 (kicad_sch
-	(version 20250114)
+	(version 20260306)
 	(generator "eeschema")
-	(generator_version "9.0")
+	(generator_version "10.0")
 	(paper "A3")
 	(title_block
