File: mcu.kicad_sch (KiCad schematic)
At the start: 39 parts, among them U400 STM32H563VGTx, X300 Q13FC1350000400, Y400 ASE-xxxMHz

Commit message: Add MX74700 lib and symbol
Other:
- title: ModuCard BM STM32H562VGT6 -> ModuCard 3 BM STM32H562VGT6
Changed lines of the file:
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@@
 	(paper "A3")
 	(title_block
-		(title "ModuCard BM STM32H562VGT6")
+		(title "ModuCard 3 BM STM32H562VGT6")
 		(date "2025-04-18")
-		(rev "1.1.1")
+		(rev "1.2.1")
 		(company "KoNaR")
-		(comment 1 "Base project authors: Dominik Pluta, Artem Horiunov")
+		(comment 1 "Base project authors: Dominik Pluta, Artem Horiunov, Maciej Chodowiec")
 		(comment 2 "Project author: <author>")
 	)
